File: mexa_badge_defcon25.sch (KiCad schematic (older format))
At the start: 6 parts

Commit message: Add Schematic
Parts:
- removed D? (x4): 1655, FCI_1655, symbol 1655
- removed U?: ESP-12E, symbol ESP-12E
- added BZ?: Buzzer, symbol Buzzer
- added C?: 4.7uF, Capacitors_SMD:C_0805_HandSoldering, symbol C
- added C? (x2): 10uF, Capacitors_SMD:C_0805_HandSoldering, symbol C
- added C?: 1.0uF, Capacitors_SMD:C_0805_HandSoldering, symbol C
- added C? (x5): 0.1uF, symbol C_Small
- added D?: LED, LEDs:LED-0805, symbol LED
- added D?: MBR120, Diodes_SMD:SOD-123, symbol ZENER
- added D?: LED, LEDs:LED-0603, symbol LED
- added D? (x2): 1N4148, Diodes_SMD:SOD-323, symbol D
- added D? (x4): 1655, FCI_1655, symbol 1655
- added P?: OLED_I2C, Socket_Strips:Socket_Strip_Straight_1x04, symbol CONN_01X04
- added P?: USB Serial, Socket_Strips:Socket_Strip_Straight_1x06, symbol CONN_01X06
- added P?: LiPo, open-project:CONN_JST-2_SMD, symbol CONN_01X02
- added P?: AUTO-PROGRAM JUMPER, Pin_Headers:Pin_Header_Straight_1x02, symbol CONN_01X02
- added P? (x2): CONN_01X10, Pin_Headers:Pin_Header_Straight_1x10, symbol CONN_01X10
- added Q?: Q_PNP_BCE, symbol Q_PNP_BCE
- added R? (x3): 1K, Resistors_SMD:R_0805_HandSoldering, symbol R
- added R? (x5): 10K, Resistors_SMD:R_0805_HandSoldering, symbol R
- added R? (x2): 3k3, Resistors_SMD:R_0805_HandSoldering, symbol R
- added R?: 220K, Resistors_SMD:R_0805_HandSoldering, symbol R
- added R?: 100K, Resistors_SMD:R_0805_HandSoldering, symbol R
- added R?: R_Small, symbol R_Small
- added U?: ESP-12E, esp:ESP-12E, symbol ESP-12E
- added U?: SPX1117, TO_SOT_Packages_SMD:SOT-223, symbol SPX1117
- added U?: MCP73831T-2ATI/OT, SOT95P300X145-5N, symbol MCP73831T-2ATI/OT
Connections:
- net labels added: +3.3V, +3V3, +BATT, ADC, ADC_IN, CH_PD, DOUT1, DOUT2, DOUT3, DOUT4, DTR, GND, GPIO0, GPIO12, GPIO13, GPIO14, GPIO15, GPIO16, GPIO2, GPIO4/SDA, GPIO5/SCL, RST, RX, TX, VCC
- wire segments 0 -> 171
- no-connect marks 0 -> 8
Other:
- note added: "10K = 100mA\n5K = 200mA\n2K = 500mA\n1K = 1000mA"
- note added: "3.3V LDO\nMax input: 15V\nMin Input: 4.4V\nMax Current: 800mA"
- note added: "ADC a 1.0V,\narreglo de resistencias \npara 3.3v"
- note added: "ADC_FIX"
- note added: "ESP8266 + AUTORESET"
- note added: "Es necesario quitar el jumper\npara Serial Terminal Debbuging"
- note added: "Features:\nNeopixel\nESP8266\nUSB+FTDI\nCargador bateria lipo\nSensor capacitivo*\nbotones\nBuzzer melodia*\n"
- note added: "HEADERS"
- note added: "LiPo Charging"
- note added: "NEOPIXEL"
- note added: "PANTALLA OLED"
- note added: "POWER AND FILTERING"
- note added: "USB-Serial"
- note added: "VCC: 3.5v to 5.3"
- note removed: "Features:\nNeopixel\nESP8266\nUSB+FTDI\nCargador bateria lipo\nSensor capacitivo*\nbotones\n"
- moved on the sheet: D?
