File: mexa_badge_defcon25.sch (KiCad schematic (older format))
At the start: 43 parts

Commit message: version 0.1
Parts:
- removed D? (x5): 1655, FCI_1655, symbol 1655
- removed U?: MCP73831T-2ATI/OT, SOT95P300X145-5N, symbol MCP73831T-2ATI/OT
- added LED1, LED2, LED3, LED4, LED5: MADW__WS2812B, symbol MADW__WS2812B
- added SW1, SW2: SW_PUSH, symbol SW_PUSH
- added U2: MCP73831, symbol MCP73831
- gave numbers to parts that had none: 37
Other:
- note added: "BUZZER"
- note added: "Features:\nNeopixel\nESP8266\nUSB+FTDI\nCargador bateria lipo\nBuzzer melodia\n\nTODO\nBotones Control o \nSensor capacitivo*\n"
- note removed: "Features:\nNeopixel\nESP8266\nUSB+FTDI\nCargador bateria lipo\nSensor capacitivo*\nbotones\nBuzzer melodia*\n"
- moved on the sheet: C5, C6, C7, C8, C9, P6, R12, R13

Commit message: Change SDA and SCL
Parts:
- added R14, R15: 10K, Resistors_SMD:R_0805_HandSoldering, symbol R_Small
- added SW3, SW4: SW_PUSH, TIH:SW_B3U-1000P, symbol SW_PUSH
- BZ1: footprint (none) -> Buzzers_Beepers:BUZZER
- C5, C6, C7, C8, C9: footprint (none) -> Capacitors_SMD:C_0805_HandSoldering
- D1: footprint LEDs:LED-0603 -> LEDs:LED_0805
- LED1, LED2, LED3, LED4, LED5: footprint (none) -> LEDs:LED_WS2812B-PLCC4
- P2: footprint open-project:CONN_JST-2_SMD -> Socket_Strips:Socket_Strip_Straight_1x02
- P3, P4: footprint Pin_Headers:Pin_Header_Straight_1x10 -> Socket_Strips:Socket_Strip_Straight_1x10
- Q1: footprint (none) -> TO_SOT_Packages_SMD:SOT-23_Handsoldering
- R8: value R_Small -> 2.2K; footprint (none) -> Resistors_SMD:R_0805_HandSoldering
- SW1: value SW_PUSH -> SW_RESET; footprint (none) -> TIH:SW_B3U-1000P
- SW2: value SW_PUSH -> SW_BOOT; footprint (none) -> TIH:SW_B3U-1000P
- U2: footprint (none) -> TO_SOT_Packages_SMD:SOT-23-5
- U3: footprint esp:ESP-12E -> ESP8266:ESP-12E
Connections:
- net +3V3: now also R14.1, R15.1
- net GND: now also R14.2, R15.2, SW3.2, SW4.2
- net GPIO12: now also SW4.1
- net GPIO13: now also SW3.1
- net GPIO4/SDA: no longer R13.2, U3.19 (GPIO4)
- net GPIO5/SCL: no longer R12.2, U3.20 (GPIO5)
- new net SCL: R12.2, U3.20 (GPIO5)
- new net SDA: R13.2, U3.19 (GPIO4)
Other:
- note removed: "Features:\nNeopixel\nESP8266\nUSB+FTDI\nCargador bateria lipo\nBuzzer melodia\n\nTODO\nBotones Control o \nSensor capacitivo*\n"
- moved on the sheet: C1, D3, D4, P1, R1, R10, R11, R3, R7, R9, SW1, SW2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
