File: mexa_badge_defcon25.kicad_pcb (KiCad board)
At the start: 2 copper layers, 148.1 x 115.1 mm, 16 parts

Commit message: Add Sponsors
Parts:
- added G***: LOGO, TIH:electronic_cats_logo_70x60, F.Cu at (345.9, 113.8)
- added G***: LOGO, TIH:electronic_cats_logo_8x6, B.Cu at (205.1, 58.1)
- added G***: LOGO, TIH:tpx_logo, B.Cu at (205.9, 66.1)
Other:
- board text added: "Sponsors"

Commit message: Init PCB
Parts:
- removed REF** (x5): LED_WS2812B-PLCC4, LEDs:LED_WS2812B-PLCC4
- removed REF**: ESP-12E, ESP8266:ESP-12E
- added BZ1: Buzzer, Buzzers_Beepers:BUZZER, F.Cu at (196.2, 85.2)
- added C1: 1.0uF, Capacitors_SMD:C_0805_HandSoldering, B.Cu at (49.5, 45.5)
- added C2: 4.7uF, Capacitors_SMD:C_0805_HandSoldering, B.Cu at (49.8, 39.5)
- added C3: 10uF, Capacitors_SMD:C_0805_HandSoldering, B.Cu at (40.2, 50.8)
- added C4: 10uF, Capacitors_SMD:C_0805_HandSoldering, B.Cu at (47.5, 60.5)
- added C5: 0.1uF, Capacitors_SMD:C_0805_HandSoldering, F.Cu at (135.5, 73.8)
- added C6: 0.1uF, Capacitors_SMD:C_0805_HandSoldering, F.Cu at (161.0, 74.2)
- added C7: 0.1uF, Capacitors_SMD:C_0805_HandSoldering, F.Cu at (147.5, 114.0)
- added C8: 0.1uF, Capacitors_SMD:C_0805_HandSoldering, F.Cu at (136.8, 126.0)
- added C9: 0.1uF, Capacitors_SMD:C_0805_HandSoldering, F.Cu at (159.5, 126.0)
- added D1: LED, LEDs:LED_0805, B.Cu at (97.8, 79.5)
- added D2: MBR120, Diodes_SMD:SOD-123, B.Cu at (46.9, 66.0)
- added D3: 1N4148, Diodes_SMD:SOD-323, B.Cu at (56.2, 52.2)
- added D5: 1N4148, Diodes_SMD:SOD-323, F.Cu at (209.8, 65.2)
- added LED1: MADW__WS2812B, LEDs:LED_WS2812B-PLCC4, F.Cu at (135.5, 79.4)
- added LED2: MADW__WS2812B, LEDs:LED_WS2812B-PLCC4, F.Cu at (161.0, 79.8)
- added LED3: MADW__WS2812B, LEDs:LED_WS2812B-PLCC4, F.Cu at (147.5, 118.8)
- added LED4: MADW__WS2812B, LEDs:LED_WS2812B-PLCC4, F.Cu at (137.0, 131.5)
- added LED5: MADW__WS2812B, LEDs:LED_WS2812B-PLCC4, F.Cu at (159.2, 131.5)
- added P2: LiPo, Socket_Strips:Socket_Strip_Straight_1x02, B.Cu at (89.2, 85.2)
- added P3: CONN_01X10, Socket_Strips:Socket_Strip_Straight_1x10, B.Cu at (136.2, 105.8)
- added P4: CONN_01X10, Socket_Strips:Socket_Strip_Straight_1x10, B.Cu at (136.2, 100.8)
- added P5: USB Serial, Socket_Strips:Socket_Strip_Straight_1x06, B.Cu at (217.5, 60.9)
- added P6: OLED_I2C, Socket_Strips:Socket_Strip_Straight_1x04, F.Cu at (132.5, 60.8)
- added Q1: Q_PNP_BCE, TO_SOT_Packages_SMD:SOT-23_Handsoldering, B.Cu at (196.8, 76.0)
- added R1: 10K, Resistors_SMD:R_0805_HandSoldering, B.Cu at (57.4, 46.2)
- added R10: 10K, Resistors_SMD:R_0805_HandSoldering, B.Cu at (73.8, 28.8)
- added R11: 10K, Resistors_SMD:R_0805_HandSoldering, B.Cu at (79.2, 29.0)
- added R12: 3k3, Resistors_SMD:R_0805_HandSoldering, B.Cu at (85.5, 29.5)
- added R13: 3k3, Resistors_SMD:R_0805_HandSoldering, B.Cu at (85.2, 35.5)
- added R14: 10K, Resistors_SMD:R_0805_HandSoldering, B.Cu at (78.8, 35.5)
- added R15: 10K, Resistors_SMD:R_0805_HandSoldering, B.Cu at (70.8, 34.8)
- added R2: 1K, Resistors_SMD:R_0805_HandSoldering, B.Cu at (90.2, 94.0)
- added R3: 1K, Resistors_SMD:R_0805_HandSoldering, B.Cu at (54.9, 33.8)
- added R4: 10K, Resistors_SMD:R_0805_HandSoldering, B.Cu at (99.0, 93.8)
- added R5: 220K, Resistors_SMD:R_0805_HandSoldering, B.Cu at (64.2, 46.2)
- added R6: 100K, Resistors_SMD:R_0805_HandSoldering, B.Cu at (61.8, 34.0)
- added R7: 1K, Resistors_SMD:R_0805_HandSoldering, B.Cu at (63.2, 40.2)
- added R8: 2.2K, Resistors_SMD:R_0805_HandSoldering, B.Cu at (64.2, 60.5)
- added R9: 10K, Resistors_SMD:R_0805_HandSoldering, B.Cu at (67.7, 28.5)
- added SW1: SW_RESET, TIH:SW_B3U-1000P, F.Cu at (193.5, 63.2)
- added SW2: SW_BOOT, TIH:SW_B3U-1000P, F.Cu at (191.5, 78.5)
- added SW3: SW_PUSH, TIH:SW_B3U-1000P, F.Cu at (116.0, 68.8)
- added SW4: SW_PUSH, TIH:SW_B3U-1000P, F.Cu at (115.8, 75.8)
- added U1: SPX1117, TO_SOT_Packages_SMD:SOT-223, B.Cu at (109.8, 87.8)
- added U2: MCP73831, TO_SOT_Packages_SMD:SOT-23-5, B.Cu at (97.8, 86.5)
- added U3: ESP-12E, ESP8266:ESP-12E, F.Cu at (140.5, 32.2)
- moved G*** 0.50 mm to (205.5, 65.8)
Other:
- outline, holes or cut-outs redrawn
- board text added: "DEFCON25"

Commit message: Pre acomodo
Parts:
- moved C1 146.0 mm to (195.0, 57.2)
- moved R3 136.6 mm to (186.0, 72.0)
- moved D3 133.2 mm to (186.0, 82.0), turned to 180 degrees
- moved R1 132.4 mm to (189.2, 57.2)
- moved R8 124.3 mm to (187.5, 76.2)
- moved R7 99.1 mm to (162.2, 36.0)
- moved R9 97.8 mm to (164.7, 41.2)
- moved R10 92.2 mm to (164.2, 46.5)
- moved R11 88.6 mm to (164.8, 51.8)
- moved R6 70.9 mm to (131.8, 45.0)
- moved R5 60.1 mm to (124.2, 45.0)
- moved D2 59.3 mm to (104.2, 80.8), turned to 90 degrees
- moved R15 55.0 mm to (108.0, 75.2)
- moved C4 51.9 mm to (93.0, 85.5), turned to 90 degrees
- moved C3 49.2 mm to (88.2, 61.5)
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Changed lines of the file:
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@@
   )
   (module Capacitors_SMD:C_0805_HandSoldering (layer B.Cu)
-    (at 49.5 45.5)
+    (at 195 57.25)
     (descr "Capacitor SMD 0805, hand soldering")
     (tags "capacitor 0805")
@@
   )
   (module Capacitors_SMD:C_0805_HandSoldering (layer B.Cu)
-    (at 49.75 39.5)
+    (at 82 70.25)
     (descr "Capacitor SMD 0805, hand soldering")
     (tags "capacitor 0805")
@@
   )
   (module Capacitors_SMD:C_0805_HandSoldering (layer B.Cu)
-    (at 40.25 50.75)
+    (at 88.25 61.5)
     (descr "Capacitor SMD 0805, hand soldering")
     (tags "capacitor 0805")
@@
   )
   (module Capacitors_SMD:C_0805_HandSoldering (layer B.Cu)
-    (at 47.5 60.5)
+    (at 93 85.5 90)
     (descr "Capacitor SMD 0805, hand soldering")
     (tags "capacitor 0805")
     (attr smd)
-    (fp_text reference C4 (at 0 2.1) (layer B.SilkS)
-      (effects (font (size 1 1) (thickness 0.15)) (justify mirror))
-    )
-    (fp_text value 10uF (at 0 -2.1) (layer B.Fab)
+    (fp_text reference C4 (at 0 2.1 90) (layer B.SilkS)
+      (effects (font (size 1 1) (thickness 0.15)) (justify mirror))
+    )
+    (fp_text value 10uF (at 0 -2.1 90) (layer B.Fab)
       (effects (font (size 1 1) (thickness 0.15)) (justify mirror))
     )
@@
     (fp_line (start 0.5 0.85) (end -0.5 0.85) (layer B.SilkS) (width 0.15))
     (fp_line (start -0.5 -0.85) (end 0.5 -0.85) (layer B.SilkS) (width 0.15))
-    (pad 1 smd rect (at -1.25 0) (size 1.5 1.25) (layers B.Cu B.Paste B.Mask)
+    (pad 1 smd rect (at -1.25 0 90) (size 1.5 1.25) (layers B.Cu B.Paste B.Mask)
       (net 7 +BATT))
-    (pad 2 smd rect (at 1.25 0) (size 1.5 1.25) (layers B.Cu B.Paste B.Mask)
+    (pad 2 smd rect (at 1.25 0 90) (size 1.5 1.25) (layers B.Cu B.Paste B.Mask)
       (net 1 GND))
     (model Capacitors_SMD.3dshapes/C_0805_HandSoldering.wrl
@@
   )
   (module Diodes_SMD:SOD-123 (layer B.Cu)
-    (at 46.85 66)
+    (at 104.25 80.75 90)
     (descr SOD-123)
     (tags SOD-123)
     (attr smd)
-    (fp_text reference D2 (at 0 2) (layer B.SilkS)
-      (effects (font (size 1 1) (thickness 0.15)) (justify mirror))
-    )
-    (fp_text value MBR120 (at 0 -2.1) (layer B.Fab)
+    (fp_text reference D2 (at 0 2 90) (layer B.SilkS)
+      (effects (font (size 1 1) (thickness 0.15)) (justify mirror))
+    )
+    (fp_text value MBR120 (at 0 -2.1 90) (layer B.Fab)
       (effects (font (size 1 1) (thickness 0.15)) (justify mirror))
     )
@@
     (fp_line (start -2.25 -1) (end 1.65 -1) (layer B.SilkS) (width 0.12))
     (fp_line (start -2.25 1) (end 1.65 1) (layer B.SilkS) (width 0.12))
-    (pad 1 smd rect (at -1.65 0) (size 0.9 1.2) (layers B.Cu B.Paste B.Mask)
+    (pad 1 smd rect (at -1.65 0 90) (size 0.9 1.2) (layers B.Cu B.Paste B.Mask)
       (net 5 VCC))
-    (pad 2 smd rect (at 1.65 0) (size 0.9 1.2) (layers B.Cu B.Paste B.Mask)
+    (pad 2 smd rect (at 1.65 0 90) (size 0.9 1.2) (layers B.Cu B.Paste B.Mask)
       (net 7 +BATT))
     (model ${KISYS3DMOD}/Diodes_SMD.3dshapes/SOD-123.wrl
@@
   )
   (module Diodes_SMD:SOD-323 (layer B.Cu)
-    (at 56.2 52.25)
+    (at 186 82 180)
     (descr SOD-323)
     (tags SOD-323)
     (attr smd)
-    (fp_text reference D3 (at 0 1.85) (layer B.SilkS)
-      (effects (font (size 1 1) (thickness 0.15)) (justify mirror))
-    )
-    (fp_text value 1N4148 (at 0.1 -1.9) (layer B.Fab)
+    (fp_text reference D3 (at 0 1.85 180) (layer B.SilkS)
+      (effects (font (size 1 1) (thickness 0.15)) (justify mirror))
+    )
+    (fp_text value 1N4148 (at 0.1 -1.9 180) (layer B.Fab)
       (effects (font (size 1 1) (thickness 0.15)) (justify mirror))
     )
@@
     (fp_line (start -1.5 -0.85) (end 1.05 -0.85) (layer B.SilkS) (width 0.12))
     (fp_line (start -1.5 0.85) (end 1.05 0.85) (layer B.SilkS) (width 0.12))
-    (pad 1 smd rect (at -1.05 0) (size 0.6 0.45) (layers B.Cu B.Paste B.Mask)
+    (pad 1 smd rect (at -1.05 0 180) (size 0.6 0.45) (layers B.Cu B.Paste B.Mask)
       (net 9 "Net-(D3-Pad1)"))
-    (pad 2 smd rect (at 1.05 0) (size 0.6 0.45) (layers B.Cu B.Paste B.Mask)
+    (pad 2 smd rect (at 1.05 0 180) (size 0.6 0.45) (layers B.Cu B.Paste B.Mask)
       (net 10 /GPIO0))
     (model Diodes_SMD.3dshapes/SOD-323.wrl
@@
   )
   (module Socket_Strips:Socket_Strip_Straight_1x02 (layer B.Cu)
-    (at 89.25 85.25)
+    (at 84.46 84.75)
     (descr "Through hole socket strip")
     (tags "socket strip")
@@
   )
   (module Resistors_SMD:R_0805_HandSoldering (layer B.Cu)
-    (at 57.35 46.25)
+    (at 189.25 57.25)
     (descr "Resistor SMD 0805, hand soldering")
     (tags "resistor 0805")
@@
   )
   (module Resistors_SMD:R_0805_HandSoldering (layer B.Cu)
-    (at 90.25 94)
+    (at 90.5 80.75)
     (descr "Resistor SMD 0805, hand soldering")
     (tags "resistor 0805")
@@
   )
   (module Resistors_SMD:R_0805_HandSoldering (layer B.Cu)
-    (at 54.9 33.75)
+    (at 186 72)
     (descr "Resistor SMD 0805, hand soldering")
     (tags "resistor 0805")
@@
   )
   (module Resistors_SMD:R_0805_HandSoldering (layer B.Cu)
-    (at 99 93.75)
+    (at 97.75 90.75)
     (descr "Resistor SMD 0805, hand soldering")
     (tags "resistor 0805")
@@
   )
   (module Resistors_SMD:R_0805_HandSoldering (layer B.Cu)
-    (at 64.15 46.25)
+    (at 124.25 45)
     (descr "Resistor SMD 0805, hand soldering")
     (tags "resistor 0805")
@@
   )
   (module Resistors_SMD:R_0805_HandSoldering (layer B.Cu)
-    (at 61.75 34)
+    (at 131.75 45)
     (descr "Resistor SMD 0805, hand soldering")
     (tags "resistor 0805")
@@
   )
   (module Resistors_SMD:R_0805_HandSoldering (layer B.Cu)
-    (at 63.25 40.25)
+    (at 162.25 36)
     (descr "Resistor SMD 0805, hand soldering")
     (tags "resistor 0805")
@@
   )
   (module Resistors_SMD:R_0805_HandSoldering (layer B.Cu)
-    (at 64.25 60.5)
+    (at 187.5 76.25)
     (descr "Resistor SMD 0805, hand soldering")
     (tags "resistor 0805")
@@
   )
   (module Resistors_SMD:R_0805_HandSoldering (layer B.Cu)
-    (at 67.65 28.5)
+    (at 164.65 41.25)
     (descr "Resistor SMD 0805, hand soldering")
     (tags "resistor 0805")
@@
   )
   (module Resistors_SMD:R_0805_HandSoldering (layer B.Cu)
-    (at 73.75 28.75)
+    (at 164.25 46.5)
     (descr "Resistor SMD 0805, hand soldering")
     (tags "resistor 0805")
@@
   )
   (module Resistors_SMD:R_0805_HandSoldering (layer B.Cu)
-    (at 79.15 29)
+    (at 164.75 51.75)
     (descr "Resistor SMD 0805, hand soldering")
     (tags "resistor 0805")
@@
   )
   (module Resistors_SMD:R_0805_HandSoldering (layer B.Cu)
-    (at 85.5 29.5)
+    (at 126 54.5)
     (descr "Resistor SMD 0805, hand soldering")
     (tags "resistor 0805")
@@
   )
   (module Resistors_SMD:R_0805_HandSoldering (layer B.Cu)
-    (at 85.15 35.5)
+    (at 125.65 60.5)
     (descr "Resistor SMD 0805, hand soldering")
     (tags "resistor 0805")
@@
   )
   (module Resistors_SMD:R_0805_HandSoldering (layer B.Cu)
-    (at 78.75 35.5)
+    (at 108 68.75)
     (descr "Resistor SMD 0805, hand soldering")
     (tags "resistor 0805")
@@
   )
   (module Resistors_SMD:R_0805_HandSoldering (layer B.Cu)
-    (at 70.75 34.75)
+    (at 108 75.25)
     (descr "Resistor SMD 0805, hand soldering")
     (tags "resistor 0805")
@@
   )
   (module TO_SOT_Packages_SMD:SOT-223 (layer B.Cu)
-    (at 109.75 87.75)
+    (at 90.5 69.25)
     (descr "module CMS SOT223 4 pins")
     (tags "CMS SOT")
@@
   )
   (module TO_SOT_Packages_SMD:SOT-23-5 (layer B.Cu)
-    (at 97.75 86.5)
+    (at 98 85)
     (descr "5-pin SOT23 package")
     (tags SOT-23-5)

Commit message: fix ways
Parts:
- moved R10 32.3 mm to (132.0, 48.0)
- moved D1 13.3 mm to (97.2, 92.8)
- moved D2 9.85 mm to (94.4, 81.0), turned to 180 degrees
- moved R2 9.81 mm to (94.4, 89.8), turned to 180 degrees
- moved C3 8.81 mm to (83.2, 68.8), turned to 270 degrees
- moved R5 8.07 mm to (132.0, 42.8)
- moved R11 7.71 mm to (160.6, 45.2)
- moved R9 7.63 mm to (160.7, 47.8), turned to 180 degrees
- moved R7 6.95 mm to (160.6, 42.8), turned to 180 degrees
- moved D3 6.14 mm to (184.5, 76.0), turned to 270 degrees
- moved R3 4.50 mm to (189.9, 74.2), turned to 180 degrees
- moved C2 2.70 mm to (79.8, 68.8), turned to 270 degrees
- moved R4 2.55 mm to (100.1, 89.8)
- moved R8 2.47 mm to (189.8, 77.0), turned to 180 degrees
- moved U3 1.03 mm to (139.5, 32.0)
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Routing:
- net VCC: track 0.00 -> 16.9 mm
- net +BATT: track 0.00 -> 6.88 mm
- net Net-(R4-Pad2): track 0.00 -> 5.86 mm
- net Net-(D1-Pad1): track 0.00 -> 5.74 mm
- net +3V3: track 0.00 -> 5.26 mm
- net Net-(R2-Pad1): track 0.00 -> 4.28 mm
Other:
- net class Default: trace_width 0.25 -> 0.3
- net class Vcc added: clearance 0.2, trace_width 0.5, via_dia 0.8, via_drill 0.6
